File: photon-sensor-board.sch (KiCad schematic (older format))
At the start: 3 parts, among them U1 PHOTON, U2 DS18B20

Commit message: Some adjustments
Connections:
- net at R1.2, U2.2 (DQ): now also U1.13 (D0); no longer U1.14 (D1)
Changed lines of the file:
@@
 NoConn ~ 6500 4400
 NoConn ~ 6500 4500
-NoConn ~ 6500 4700
+NoConn ~ 6500 4600
 NoConn ~ 6500 3500
 NoConn ~ 6500 3400
@@
 	5600 3100 4350 3100
 Connection ~ 4600 3500
-Wire Wire Line
-	6600 4600 6500 4600
 Connection ~ 6600 3150
 Wire Wire Line
-	6600 3150 6600 4600
+	6600 3150 6600 4700
 Wire Wire Line
 	5950 3150 5950 2650
@@
 Wire Wire Line
 	5800 2650 5800 3200
+Wire Wire Line
+	6600 4700 6500 4700
 $EndSCHEMATC
