File: photon-sensor-board.kicad_pcb (KiCad board)
At the start: 2 copper layers, 35 x 50 mm, 6 parts, among them M1 MountingHole_2-5mm, M2 MountingHole_2-5mm, U1 PHOTON, U2 DS18B20

Commit message: Exported v1.2
Routing:
- added copper zone on B.Cu, net GND
Other:
- board text added: "Coredump Rapperswil www.coredump.ch"
- board text added: "Photon Sensor Board v1.2 2015"
- board text removed: "Photon Sensor Board v1.1 2015"
Changed lines of the file:
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@@
-(kicad_pcb (version 4) (host pcbnew "(2015-10-02 BZR 6241)-product")
+(kicad_pcb (version 4) (host pcbnew "(2015-11-24 BZR 6329, Git e511afd)-product")
   (general
     (links 6)
     (no_connects 0)
-    (area 108.22388 67.32988 150.850584 124.744464)
+    (area 110.029999 69.041999 145.130001 119.142001)
     (thickness 1.6)
-    (drawings 6)
+    (drawings 7)
     (tracks 22)
     (zones 0)
@@
   )
   (layers
-    (0 F.Cu signal)
-    (31 B.Cu signal hide)
-    (32 B.Adhes user hide)
+    (0 F.Cu signal hide)
+    (31 B.Cu signal)
+    (32 B.Adhes user)
     (33 F.Adhes user)
-    (34 B.Paste user hide)
+    (34 B.Paste user)
     (35 F.Paste user)
-    (36 B.SilkS user hide)
+    (36 B.SilkS user)
     (37 F.SilkS user)
-    (38 B.Mask user hide)
+    (38 B.Mask user)
     (39 F.Mask user)
-    (40 Dwgs.User user)
-    (41 Cmts.User user)
+    (40 Dwgs.User user hide)
+    (41 Cmts.User user hide)
     (42 Eco1.User user hide)
     (43 Eco2.User user hide)
@@
     (last_trace_width 0.508)
     (trace_clearance 0.381)
-    (zone_clearance 0.381)
+    (zone_clearance 0.508)
     (zone_45_only no)
     (trace_min 0.508)
@@
     (visible_elements FFFCFFBF)
     (pcbplotparams
-      (layerselection 0x00030_80000001)
+      (layerselection 0x010f0_80000001)
       (usegerberextensions true)
       (excludeedgelayer true)
@@
       (psnegative false)
       (psa4output false)
-      (plotreference true)
-      (plotvalue true)
+      (plotreference false)
+      (plotvalue false)
       (plotinvisibletext false)
       (padsonsilk false)
@@
       (drillshape 0)
       (scaleselection 1)
-      (outputdirectory export/v1.0/))
+      (outputdirectory export/v1.2/))
   )
   (net 0 "")
@@
     )
   )
-  (gr_text "Photon Sensor Board v1.1 2015" (at 142.494 90.424 270) (layer F.Mask)
+  (gr_text "Coredump Rapperswil\nwww.coredump.ch" (at 142.24 113.03) (layer B.Mask)
+    (effects (font (size 1.5 1.5) (thickness 0.3)) (justify left mirror))
+  )
+  (gr_text "Photon Sensor Board v1.2 2015" (at 142.494 90.424 270) (layer F.Mask)
     (effects (font (size 1.2 1.2) (thickness 0.2)))
   )
@@
       )
     )
+  )
+  (zone (net 1) (net_name GND) (layer B.Cu) (hatch edge 0.508)
+    (connect_pads (clearance 0.508))
+    (min_thickness 0.254)
+    (fill yes (arc_segments 16) (thermal_gap 0.508) (thermal_bridge_width 0.508))
+    (polygon
+      (pts
+        (xy 107.95 67.31) (xy 147.32 67.31) (xy 147.32 120.65) (xy 107.95 120.65)
+      )
+    )
